Commit message: Tidy up the URDF, add a macro for the internal camera structure to reduce copypasta.  Order of the cameras is verified; 0 is forward, 1-4 are in-order moving clockiwse when viewed from above.

File: urdf/omni_60.urdf.xacro (robot description, xacro)
@@ -25,70 +25,20 @@
       <xacro:insert_block name="origin" />
     </joint>
-    <!--
-      The 5 cameras are arrayed radially, so define 2 links per camera: one in the middle with the correct yaw
-      and a second for the actual image frame.  This lets us basically use polar coordinates, instead of
-      caluclating XYZ transforms for each frame
-    -->
-    <!-- TODO double-check which way around the lenses are enumerated on an actual camera -->
-    <link name="${name}_camera1_link"/>
-    <link name="${name}_camera2_link"/>
-    <link name="${name}_camera3_link"/>
-    <link name="${name}_camera4_link"/>
-    <link name="${name}_camera5_link"/>
-    <link name="${name}_camera1_internal_link"/>
-    <link name="${name}_camera2_internal_link"/>
-    <link name="${name}_camera3_internal_link"/>
-    <link name="${name}_camera4_internal_link"/>
-    <link name="${name}_camera5_internal_link"/>
-    <joint name="${name}_camera3_orientation_joint" type="fixed">
-      <parent link="${name}_base_link" />
-      <child link="${name}_camera3_internal_link" />
+    <include filename="$(find occam_ros)/urdf/include/omni_sub_camera.urdf.xacro" />
+    <xacro:omni_sub_camera prefix="${name}_camera0" parent="${name}_base_link">
       <origin xyz="0 0 0.026" rpy="0 0 0" />
-    </joint>
-    <joint name="${name}_camera2_orientation_joint" type="fixed">
-      <parent link="${name}_camera3_internal_link" />
-      <child link="${name}_camera2_internal_link" />
-      <origin xyz="0 0 0" rpy="0 0 ${2*pi/5}" />
-    </joint>
-    <joint name="${name}_camera1_orientation_joint" type="fixed">
-      <parent link="${name}_camera3_internal_link" />
-      <child link="${name}_camera1_internal_link" />
-      <origin xyz="0 0 0" rpy="0 0 ${4*pi/5}" />
-    </joint>
-    <joint name="${name}_camera4_orientation_joint" type="fixed">
-      <parent link="${name}_camera3_internal_link" />
-      <child link="${name}_camera4_internal_link" />
-      <origin xyz="0 0 0" rpy="0 0 -${2*pi/5}" />
-    </joint>
-    <joint name="${name}_camera5_orientation_joint" type="fixed">
-      <parent link="${name}_camera3_internal_link" />
-      <child link="${name}_camera5_internal_link" />
-      <origin xyz="0 0 0" rpy="0 0 -${4*pi/5}" />
-    </joint>
-    <joint name="${name}_camera3_joint" type="fixed">
-      <parent link="${name}_camera3_internal_link" />
-      <child link="${name}_camera3_link" />
-      <origin xyz="0.05225 0 0" rpy="0 0 0" />
-    </joint>
-    <joint name="${name}_camera2_joint" type="fixed">
-      <parent link="${name}_camera2_internal_link" />
-      <child link="${name}_camera2_link" />
-      <origin xyz="0.05225 0 0" rpy="0 0 0" />
-    </joint>
-    <joint name="${name}_camera1_joint" type="fixed">
-      <parent link="${name}_camera1_internal_link" />
-      <child link="${name}_camera1_link" />
-      <origin xyz="0.05225 0 0" rpy="0 0 0" />
-    </joint>
-    <joint name="${name}_camera4_joint" type="fixed">
-      <parent link="${name}_camera4_internal_link" />
-      <child link="${name}_camera4_link" />
-      <origin xyz="0.05225 0 0" rpy="0 0 0" />
-    </joint>
-    <joint name="${name}_camera5_joint" type="fixed">
-      <parent link="${name}_camera5_internal_link" />
-      <child link="${name}_camera5_link" />
-      <origin xyz="0.05225 0 0" rpy="0 0 0" />
-    </joint>
+    </xacro:omni_sub_camera>
+    <xacro:omni_sub_camera prefix="${name}_camera1" parent="${name}_base_link">
+      <origin xyz="0 0 0.026" rpy="0 0 -${2*pi/5}" />
+    </xacro:omni_sub_camera>
+    <xacro:omni_sub_camera prefix="${name}_camera2" parent="${name}_base_link">
+      <origin xyz="0 0 0.026" rpy="0 0 -${4*pi/5}" />
+    </xacro:omni_sub_camera>
+    <xacro:omni_sub_camera prefix="${name}_camera3" parent="${name}_base_link">
+      <origin xyz="0 0 0.026" rpy="0 0 ${4*pi/5}" />
+    </xacro:omni_sub_camera>
+    <xacro:omni_sub_camera prefix="${name}_camera4" parent="${name}_base_link">
+      <origin xyz="0 0 0.026" rpy="0 0 ${2*pi/5}" />
+    </xacro:omni_sub_camera>
   </xacro:macro>
 </robot>

Commit message: Remove references to ${pi}, replace with the explicit number; pi is defined in the Jackal URDF, but doesn't exist on other platforms.

File: urdf/omni_60.urdf.xacro (robot description, xacro)
@@ -7,5 +7,5 @@
           <mesh filename="package://occam_ros/meshes/omni_60.stl" />
         </geometry>
-        <origin xyz="0 0 0" rpy="${pi/2} 0 -${pi/2}" />
+        <origin xyz="0 0 0" rpy="${3.141592653589793/2} 0 -${3.141592653589793/2}" />
         <material name="navy">
           <color rgba="0.1 0.1 0.7 1" />
@@ -30,14 +30,14 @@
     </xacro:omni_sub_camera>
     <xacro:omni_sub_camera prefix="${name}_camera1" parent="${name}_base_link">
-      <origin xyz="0 0 0.026" rpy="0 0 -${2*pi/5}" />
+      <origin xyz="0 0 0.026" rpy="0 0 -${2*3.141592653589793/5}" />
     </xacro:omni_sub_camera>
     <xacro:omni_sub_camera prefix="${name}_camera2" parent="${name}_base_link">
-      <origin xyz="0 0 0.026" rpy="0 0 -${4*pi/5}" />
+      <origin xyz="0 0 0.026" rpy="0 0 -${4*3.141592653589793/5}" />
     </xacro:omni_sub_camera>
     <xacro:omni_sub_camera prefix="${name}_camera3" parent="${name}_base_link">
-      <origin xyz="0 0 0.026" rpy="0 0 ${4*pi/5}" />
+      <origin xyz="0 0 0.026" rpy="0 0 ${4*3.141592653589793/5}" />
     </xacro:omni_sub_camera>
     <xacro:omni_sub_camera prefix="${name}_camera4" parent="${name}_base_link">
-      <origin xyz="0 0 0.026" rpy="0 0 ${2*pi/5}" />
+      <origin xyz="0 0 0.026" rpy="0 0 ${2*3.141592653589793/5}" />
     </xacro:omni_sub_camera>
   </xacro:macro>

Commit message: Update the STL so the orientation is correct, remove the roll/yaw transformations in the URDF

File: urdf/omni_60.urdf.xacro (robot description, xacro)
@@ -7,5 +7,5 @@
           <mesh filename="package://occam_ros/meshes/omni_60.stl" />
         </geometry>
-        <origin xyz="0 0 0" rpy="${3.141592653589793/2} 0 -${3.141592653589793/2}" />
+        <origin xyz="0 0 0" rpy="0 0 0" />
         <material name="navy">
           <color rgba="0.1 0.1 0.7 1" />
